Commit message: added reduced urdf

File: ouster_os1_64/urdf/example_robot.urdf.xacro (robot description, xacro)
@@ -1,9 +1,9 @@
 <?xml version="1.0"?>
-<robot xmlns:xacro="http://ros.org/wiki/xacro" name="example_robot">
+<robot xmlns:xacro="http://ros.org/wiki/xacro" name="os1_64">
   <!-- Base Footprint -->
   <link name="base_footprint_link" />
-  <xacro:include filename="$(find ouster_os1_64)/urdf/os1_64.urdf.xacro"/>
-  <xacro:os1_64 parent="base_footprint" name="ouster" prefix="/os1_cloud_node" hz="10" samples="512">
+  <xacro:include filename="$(find ouster_os1_64)/urdf/os1_64_simple.urdf.xacro"/>
+  <!--xacro:os1_64 parent="base_footprint" name="ouster" prefix="/os1_cloud_node" hz="10" samples="512">
     <origin xyz="0 0 0" rpy="0 0 0" />
-  </xacro:os1_64>
+  </xacro:os1_64-->
 </robot>

File: ouster_os1_64/urdf/os1_64.urdf.xacro (robot description, xacro)
@@ -49,5 +49,15 @@
       <child link="${name}_lidar"/>
     </joint>
+    <!-- Fix w.r.t. world by adding a fixed link -->
+    <!--
+    <link name="world" />
+    <joint name="world_joint"  type="fixed">
+        <origin xyz="0 0 1." rpy="0 0 0" />
+        <parent link="world"/>
+        <child link="base_footprint_link"/>
+    </joint>
+    -->
     <gazebo reference="${name}_lidar">
+      <static>true</static>
       <sensor type="${gpu_str}ray" name="${name}_lidar">
         <pose>0 0 0 0 0 0</pose>
