Commit message: Update for SOF_1537

File: ouster_os1_64/urdf/os1_64.urdf.xacro (robot description, xacro)
@@ -3,5 +3,5 @@
 <robot xmlns:xacro="http://ros.org/wiki/xacro" name="os1_64">
   <xacro:property name="PI" value="3.1415926535897931"/>
-  <xacro:macro name="os1_64" params="*origin parent:=base name:=ouster reduced:=true prefix:=/os1_cloud_node hz:=10 samples:=512 min_range:=0.8 max_range:=100 noise:=0.008 min_angle_v:=-16.6 max_angle_v:=16.6 gpu:=false">
+  <xacro:macro name="os1_64" params="*origin parent:=base name:=ouster reduced:=true prefix:=/os1_cloud_node hz:=10 samples:=512 min_range:=0.8 max_range:=100 noise:=0.008 min_angle_v:=-22.5 max_angle_v:=22.5 gpu:=false">
     <!-- Conditional properties -->
     <xacro:if value="${reduced}">
@@ -24,15 +24,15 @@
     <link name="${name}_sensor">
       <inertial>
-        <mass value="0.425"/>
+        <mass value="0.000001"/>
         <origin xyz="0 0 0.03675" rpy="0 0 0" />
         <inertia ixx="0.000308429" ixy="0" ixz="0"
                  iyy="0.000308429" iyz="0" izz="0.00034589"/>
       </inertial>
-      <collision name="lidar_collision">
+      <!-- <collision name="lidar_collision">
         <origin xyz="0 0 0.03675" rpy="0 0 0" />
         <geometry>
           <cylinder radius="0.04350" length="0.07350"/>
         </geometry>
-      </collision>
+      </collision> -->
       <visual name="lidar_visual">
         <origin xyz="0 0 0" rpy="0 0 0"/>
@@ -48,16 +48,7 @@
       <parent link="${name}_sensor"/>
       <child link="${name}_lidar"/>
+      <origin xyz="0 0 0.037" rpy="0 0 ${PI}" />
     </joint>
-    <!-- Fix w.r.t. world by adding a fixed link -->
-    <!--
-    <link name="world" />
-    <joint name="world_joint"  type="fixed">
-        <origin xyz="0 0 1." rpy="0 0 0" />
-        <parent link="world"/>
-        <child link="base_footprint_link"/>
-    </joint>
-    -->
     <gazebo reference="${name}_lidar">
-      <static>true</static>
       <sensor type="${gpu_str}ray" name="${name}_lidar">
         <pose>0 0 0 0 0 0</pose>
